Commit message: Commit from theconstructsim to fiz gazebo

File: ovis_description/urdf/ovis_standalone copy.xacro (robot description, xacro)
@@ -41,5 +41,5 @@
     <limit effort="40" lower="-12.5663706144" upper="12.5663706144" velocity="0.628318530718" />
     <origin rpy="0 0 0" xyz="0 0 0.051" />
-    <dynamics damping="0.5" friction="0.01" />
+    <dynamics damping="0.0" friction="0.0" />
   </joint>
   <link name="ovis_link_1">
@@ -69,5 +69,5 @@
     <limit effort="80" lower="-1.57079632679" upper="1.57079632679" velocity="0.628318530718" />
     <origin rpy="1.57079632679 0 0" xyz="0 0 0.0889" />
-    <dynamics damping="0.5" friction="0.01" />
+    <dynamics damping="0.0" friction="0.0" />
   </joint>
   <link name="ovis_link_2">
@@ -97,5 +97,5 @@
     <limit effort="40" lower="-1.57079632679" upper="1.57079632679" velocity="0.628318530718" />
     <origin rpy="0 0 1.57079632679" xyz="0 0.465 0" />
-    <dynamics damping="0.5" friction="0.01" />
+    <dynamics damping="0.0" friction="0.0" />
   </joint>
   <link name="ovis_link_3">
@@ -125,5 +125,5 @@
     <limit effort="20" lower="-12.5663706144" upper="12.5663706144" velocity="0.837758040957" />
     <origin rpy="0 0 0" xyz="0.0889 0.047625 0" />
-    <dynamics damping="0.5" friction="0.01" />
+    <dynamics damping="0.0" friction="0.0" />
   </joint>
   <link name="ovis_link_4">
@@ -153,5 +153,5 @@
       <limit effort="20" lower="-1.57079632679" upper="1.57079632679" velocity="0.837758040957" />
       <origin rpy="0 0 0" xyz="0 0.265 0" />
-      <dynamics damping="0.5" friction="0.01" />
+      <dynamics damping="0.0" friction="0.0" />
   </joint>
   <link name="ovis_link_5">
@@ -181,5 +181,5 @@
         <limit effort="20" lower="-6.28318530718" upper="6.28318530718" velocity="0.837758040957" />
         <origin rpy="1.57079632679 1.57079632679 0" xyz="0 0.0762 0" />
-        <dynamics damping="0.5" friction="0.01" />
+        <dynamics damping="0.0" friction="0.0" />
   </joint>
   <link name="ovis_link_6">

File: ovis_moveit_config/config/ovis_gazebo.ros2_control.xacro (robot description, xacro)
@@ -1,6 +1,5 @@
 <?xml version="1.0"?>
 <robot xmlns:xacro="http://www.ros.org/wiki/xacro">
-    <xacro:macro name="ovis_ros2_control" params="name initial_positions_file">
-        <xacro:property name="initial_positions" value="${load_yaml(initial_positions_file)['initial_positions']}"/>
+    <xacro:macro name="ovis_ros2_control" params="name">
         <ros2_control name="${name}" type="system">
             <hardware>
@@ -10,5 +9,5 @@
                 <command_interface name="position"/>
                 <state_interface name="position">
-                  <param name="initial_value">${initial_positions['arm_joint_1']}</param>
+                  <param name="initial_value">0.0</param>
                 </state_interface>
                 <state_interface name="velocity">
@@ -19,5 +18,5 @@
                 <command_interface name="position"/>
                 <state_interface name="position">
-                  <param name="initial_value">${initial_positions['arm_joint_2']}</param>
+                  <param name="initial_value">0.0</param>
                 </state_interface>
                 <state_interface name="velocity">
@@ -28,5 +27,5 @@
                 <command_interface name="position"/>
                 <state_interface name="position">
-                  <param name="initial_value">${initial_positions['arm_joint_3']}</param>
+                  <param name="initial_value">0.0</param>
                 </state_interface>
                 <state_interface name="velocity">
@@ -37,5 +36,5 @@
                 <command_interface name="position"/>
                 <state_interface name="position">
-                  <param name="initial_value">${initial_positions['arm_joint_4']}</param>
+                  <param name="initial_value">0.0</param>
                 </state_interface>
                 <state_interface name="velocity">
@@ -46,5 +45,5 @@
                 <command_interface name="position"/>
                 <state_interface name="position">
-                  <param name="initial_value">${initial_positions['arm_joint_5']}</param>
+                  <param name="initial_value">0.0</param>
                 </state_interface>
                 <state_interface name="velocity">
@@ -55,5 +54,5 @@
                 <command_interface name="position"/>
                 <state_interface name="position">
-                  <param name="initial_value">${initial_positions['arm_joint_6']}</param>
+                  <param name="initial_value">0.0</param>
                 </state_interface>
                 <state_interface name="velocity">
@@ -64,8 +63,5 @@
         <!-- Gazebo ros2_control plugin -->
         <gazebo>
-        <plugin filename="libgazebo_ros2_control.so" name="gazebo_ros2_control}">
-            <robotSimType>gazebo_ros2_control/DefaultRobotHWSim</robotSimType>
-            <robot_param>robot_description</robot_param>
-            <robot_param_node>robot_state_publisher</robot_param_node>
+        <plugin filename="libgazebo_ros2_control.so" name="gazebo_ros2_control">
           <parameters>$(find ovis_bringup)/config/gaz_ros2_ctl_use_sim.yaml</parameters>
           <parameters>$(find ovis_moveit_config)/config/ros2_controllers.yaml</parameters>

File: ovis_moveit_config/config/ovis_gazebo.urdf.xacro (robot description, xacro)
@@ -4,7 +4,6 @@
     <!-- Import ovis urdf file -->
     <xacro:include filename="$(find ovis_description)/urdf/ovis_standalone.xacro" />
-    <xacro:include filename="$(find ovis_description)/urdf/ovis.gazebo" />
     <!-- Import control_xacro -->
     <xacro:include filename="ovis_gazebo.ros2_control.xacro" />
-    <xacro:ovis_ros2_control name="GazeboSystem" initial_positions_file="$(arg initial_positions_file)"/>
+    <xacro:ovis_ros2_control name="GazeboSystem"/>
 </robot>
